File: bm83-featherwing/bm83-featherwing.kicad_sch (KiCad schematic)
At the start: 1 part, among them U1 BM83SM1-00AA

Commit message: BM83 work
Parts:
- added C1, C2: 1uF, Capacitor_SMD:C_0805_2012Metric_Pad1.18x1.45mm_HandSolder, symbol Device:C_Small
- added C3, C4: 0.1uF, Capacitor_SMD:C_0805_2012Metric_Pad1.18x1.45mm_HandSolder, symbol Device:C_Small
- added D1, D2: PESD5V0S1BA, Diode_SMD:D_SOD-323_HandSoldering, symbol Device:D_TVS
- added D3: SMBJ10CA, Diode_SMD:D_SMB_Handsoldering, symbol Device:D_TVS
- added D4, D5: LED_Small, LED_SMD:LED_0805_2012Metric_Pad1.15x1.40mm_HandSolder, symbol Device:LED_Small
- added D6, D7: D_TVS, Diode_SMD:D_SOD-323_HandSoldering, symbol Device:D_TVS
- added J1: TOP, Footprints:RoundPinHeader_1x12, symbol Connector_Generic:Conn_01x12
- added J2: BOT, Footprints:RoundPinHeader_1x16, symbol Connector_Generic:Conn_01x16
- added J3: DX07S016JA1R1500, Footprints:JAE_DX07S016JA1R1500, symbol DX07S016JA1R1500:DX07S016JA1R1500
- added R1, R2: 5.1K, Resistor_SMD:R_0805_2012Metric_Pad1.20x1.40mm_HandSolder, symbol Device:R_Small
- added R3: 4.7K, Resistor_SMD:R_0805_2012Metric_Pad1.20x1.40mm_HandSolder, symbol Device:R_Small
- added SW1: Reset Switch, Footprints:PTS636SK25SMTRLFS, symbol Switch:SW_Push
- added SW2: Power Switch, Footprints:PTS636SK25SMTRLFS, symbol Switch:SW_Push
- added SW3: Config Switch, Footprints:PTS636SK25SMTRLFS, symbol Switch:SW_Push
Connections:
- net GND: now also C1.2, C2.2, C3.2, C4.2, D1.1 (A1), D2.1 (A1), D3.2 (A2), D6.1 (A1), D7.1 (A1), J2.13 (Pin_13), J3.1 (GND), J3.12 (GND), J3.S1 (SHIELD), J3.S2 (SHIELD), J3.S3 (SHIELD), J3.S4 (SHIELD), J3.S5 (SHIELD), J3.S6 (SHIELD), R1.1, R2.2, SW3.2
- net LRCK: now reaches U1.2 (RFS1)
- net LRCK: now also J2.9 (Pin_9)
- net ADAP_IN: now reaches U1.22 (ADAP_IN)
- net ADAP_IN: now also C1.1, D3.1 (A1), J3.11 (VBUS), J3.2 (VBUS)
- net +3V3: now reaches U1.23 (BAT_IN)
- net +3V3: now also C2.1, J2.15 (Pin_15)
- net SYS_PWR: now reaches U1.24 (SYS_PWR)
- net SYS_PWR: now also C4.1, D4.2 (A), D5.2 (A), SW2.1
- net VDD_IO: now reaches U1.25 (VDD_IO)
- net VDD_IO: now also C3.1, R3.1
- net MFB: now reaches U1.26 (PWR_(MFB))
- net MFB: now also D7.2 (A2), J1.5 (Pin_5), SW2.2
- net RXD: now reaches U1.29 (P8_6/UART_RXD)
- net RXD: now also J1.7 (Pin_7)
- net SCK: now reaches U1.3 (SCLK1)
- net SCK: now also J2.10 (Pin_10)
- net TXD: now reaches U1.30 (P8_5/UART_TXD)
- net TXD: now also J1.6 (Pin_6)
- net P3_4: now reaches U1.31 (P3_4/UART_RTS)
- net P3_4: now also SW3.1
- net LED1: now reaches U1.32 (LED1)
- net LED1: now also D4.1 (K)
- net LED2: now reaches U1.34 (LED2)
- net LED2: now also D5.1 (K)
- net USB_DM: now reaches U1.36 (DM)
- net USB_DM: now also D2.2 (A2), J3.5 (D-), J3.8 (D-)
- net USB_DP: now reaches U1.37 (DP)
- net USB_DP: now also D1.2 (A2), J3.6 (D+), J3.7 (D+)
- net SDI: now reaches U1.4 (DT1)
- net SDI: now also J2.8 (Pin_8)
- net RST_N: now reaches U1.43 (RST_N)
- net RST_N: now also D6.2 (A2), R3.2, SW1.1, SW1.2
- net MCK: now reaches U1.5 (MCLK1)
- net MCK: now also J2.3 (Pin_3)
- new net: J3.3 (CC1), R1.2
- new net: J3.9 (CC2), R2.1
- new net +3.3VA: J2.1 (Pin_1)
- no-connect marks 0 -> 50

Commit message: BM83 SPST switch
Parts:
- removed D6, D7: D_TVS, Diode_SMD:D_SOD-323_HandSoldering, symbol Device:D_TVS
- removed SW3: Config Switch, Footprints:PTS636SK25SMTRLFS, symbol Switch:SW_Push
- added SW?: SW_DIP_x01, symbol Switch:SW_DIP_x01
Connections:
- net GND: now also SW1.1, SW?.2
- net P3_4: now also SW?.1
- net RST_N: no longer SW1.1
Changed lines of the file:
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@@
   (junction (at 96.52 43.18) (diameter 0.9144) (color 0 0 0 0))
   (junction (at 229.87 54.61) (diameter 0.9144) (color 0 0 0 0))
-  (junction (at 229.87 76.2) (diameter 0.9144) (color 0 0 0 0))
   (junction (at 229.87 104.14) (diameter 0.9144) (color 0 0 0 0))
   (no_connect (at 40.64 154.94))
@@
     (stroke (width 0) (type solid) (color 0 0 0 0))
   )
-  (wire (pts (xy 224.79 76.2) (xy 229.87 76.2))
+  (wire (pts (xy 224.79 76.2) (xy 240.03 76.2))
     (stroke (width 0) (type solid) (color 0 0 0 0))
   )
@@
     (stroke (width 0) (type solid) (color 0 0 0 0))
   )
-  (wire (pts (xy 229.87 54.61) (xy 229.87 57.15))
-    (stroke (width 0) (type solid) (color 0 0 0 0))
-  )
   (wire (pts (xy 229.87 54.61) (xy 240.03 54.61))
     (stroke (width 0) (type solid) (color 0 0 0 0))
   )
-  (wire (pts (xy 229.87 76.2) (xy 229.87 78.74))
-    (stroke (width 0) (type solid) (color 0 0 0 0))
-  )
-  (wire (pts (xy 229.87 76.2) (xy 240.03 76.2))
-    (stroke (width 0) (type solid) (color 0 0 0 0))
-  )
   (wire (pts (xy 229.87 99.06) (xy 229.87 104.14))
     (stroke (width 0) (type solid) (color 0 0 0 0))
@@
     )
   )
-  (global_label "RST_N" (shape input) (at 214.63 54.61 180)
-    (effects (font (size 1.27 1.27)) (justify right))
-    (property "Intersheet References" "${INTERSHEET_REFS}" (id 0) (at 206.4717 54.5306 0)
+  (global_label "GND" (shape input) (at 214.63 54.61 180)
+    (effects (font (size 1.27 1.27)) (justify right))
+    (property "Intersheet References" "${INTERSHEET_REFS}" (id 0) (at 208.3464 54.5306 0)
       (effects (font (size 1.27 1.27)) (justify right) hide)
     )
@@
     )
   )
-  (global_label "P3_4" (shape input) (at 224.79 33.02 180)
-    (effects (font (size 1.27 1.27)) (justify right))
-    (property "Intersheet References" "${INTERSHEET_REFS}" (id 0) (at 217.7202 32.9406 0)
+  (global_label "P3_4" (shape input) (at 223.52 27.94 180)
+    (effects (font (size 1.27 1.27)) (justify right))
+    (property "Intersheet References" "${INTERSHEET_REFS}" (id 0) (at 216.4502 27.8606 0)
       (effects (font (size 1.27 1.27)) (justify right) hide)
     )
@@
     (pin "1")
   )
-  (symbol (lib_id "power:GND") (at 229.87 64.77 0) (unit 1)
-    (in_bom yes) (on_board yes)
-    (property "Reference" "#PWR0116" (id 0) (at 229.87 71.12 0)
-      (effects (font (size 1.27 1.27)) hide)
-    )
-    (property "Value" "GND" (id 1) (at 229.87 69.85 0))
-    (property "Footprint" "" (id 2) (at 229.87 64.77 0)
-      (effects (font (size 1.27 1.27)) hide)
-    )
-    (property "Datasheet" "" (id 3) (at 229.87 64.77 0)
-      (effects (font (size 1.27 1.27)) hide)
-    )
-    (pin "1")
-  )
-  (symbol (lib_id "power:GND") (at 229.87 86.36 0) (unit 1)
-    (in_bom yes) (on_board yes)
-    (property "Reference" "#PWR0115" (id 0) (at 229.87 92.71 0)
-      (effects (font (size 1.27 1.27)) hide)
-    )
-    (property "Value" "GND" (id 1) (at 229.87 91.44 0))
-    (property "Footprint" "" (id 2) (at 229.87 86.36 0)
-      (effects (font (size 1.27 1.27)) hide)
-    )
-    (property "Datasheet" "" (id 3) (at 229.87 86.36 0)
-      (effects (font (size 1.27 1.27)) hide)
-    )
-    (pin "1")
-  )
-  (symbol (lib_id "power:GND") (at 234.95 33.02 90) (unit 1)
-    (in_bom yes) (on_board yes)
-    (property "Reference" "#PWR0114" (id 0) (at 241.3 33.02 0)
-      (effects (font (size 1.27 1.27)) hide)
-    )
-    (property "Value" "GND" (id 1) (at 240.03 33.02 0))
-    (property "Footprint" "" (id 2) (at 234.95 33.02 0)
-      (effects (font (size 1.27 1.27)) hide)
-    )
-    (property "Datasheet" "" (id 3) (at 234.95 33.02 0)
+  (symbol (lib_id "power:GND") (at 238.76 27.94 90) (unit 1)
+    (in_bom yes) (on_board yes)
+    (property "Reference" "#PWR0114" (id 0) (at 245.11 27.94 0)
+      (effects (font (size 1.27 1.27)) hide)
+    )
+    (property "Value" "GND" (id 1) (at 243.84 27.94 0))
+    (property "Footprint" "" (id 2) (at 238.76 27.94 0)
+      (effects (font (size 1.27 1.27)) hide)
+    )
+    (property "Datasheet" "" (id 3) (at 238.76 27.94 0)
       (effects (font (size 1.27 1.27)) hide)
     )
@@
     (pin "2")
   )
-  (symbol (lib_id "Device:D_TVS") (at 229.87 60.96 90) (unit 1)
-    (in_bom yes) (on_board yes)
-    (property "Reference" "D6" (id 0) (at 232.41 59.69 90)
-      (effects (font (size 1.27 1.27)) (justify right))
-    )
-    (property "Value" "D_TVS" (id 1) (at 232.41 62.23 90)
-      (effects (font (size 1.27 1.27)) (justify right))
-    )
-    (property "Footprint" "Diode_SMD:D_SOD-323_HandSoldering" (id 2) (at 229.87 60.96 0)
-      (effects (font (size 1.27 1.27)) hide)
-    )
-    (property "Datasheet" "~" (id 3) (at 229.87 60.96 0)
-      (effects (font (size 1.27 1.27)) hide)
-    )
-    (pin "1")
-    (pin "2")
-  )
-  (symbol (lib_id "Device:D_TVS") (at 229.87 82.55 90) (unit 1)
-    (in_bom yes) (on_board yes)
-    (property "Reference" "D7" (id 0) (at 232.41 81.28 90)
-      (effects (font (size 1.27 1.27)) (justify right))
-    )
-    (property "Value" "D_TVS" (id 1) (at 232.41 83.82 90)
-      (effects (font (size 1.27 1.27)) (justify right))
-    )
-    (property "Footprint" "Diode_SMD:D_SOD-323_HandSoldering" (id 2) (at 229.87 82.55 0)
-      (effects (font (size 1.27 1.27)) hide)
-    )
-    (property "Datasheet" "~" (id 3) (at 229.87 82.55 0)
-      (effects (font (size 1.27 1.27)) hide)
-    )
-    (pin "1")
-    (pin "2")
-  )
   (symbol (lib_id "Switch:SW_Push") (at 219.71 54.61 0) (unit 1)
     (in_bom yes) (on_board yes)
@@
     (pin "2")
   )
-  (symbol (lib_id "Switch:SW_Push") (at 229.87 33.02 0) (unit 1)
-    (in_bom yes) (on_board yes)
-    (property "Reference" "SW3" (id 0) (at 229.87 25.4 0))
-    (property "Value" "Config Switch" (id 1) (at 229.87 27.94 0))
-    (property "Footprint" "Footprints:PTS636SK25SMTRLFS" (id 2) (at 229.87 27.94 0)
-      (effects (font (size 1.27 1.27)) hide)
-    )
-    (property "Datasheet" "~" (id 3) (at 229.87 27.94 0)
+  (symbol (lib_id "Switch:SW_DIP_x01") (at 231.14 27.94 0) (unit 1)
+    (in_bom yes) (on_board yes)
+    (property "Reference" "SW?" (id 0) (at 231.14 20.32 0))
+    (property "Value" "SW_DIP_x01" (id 1) (at 231.14 22.86 0))
+    (property "Footprint" "" (id 2) (at 231.14 27.94 0)
+      (effects (font (size 1.27 1.27)) hide)
+    )
+    (property "Datasheet" "~" (id 3) (at 231.14 27.94 0)
       (effects (font (size 1.27 1.27)) hide)
     )
@@
       (reference "#PWR0114") (unit 1) (value "GND") (footprint "")
     )
-    (path "/26f9ef42-32e7-46ac-9849-e9420d1d3995"
-      (reference "#PWR0115") (unit 1) (value "GND") (footprint "")
-    )
-    (path "/ba6cdcd0-d19b-4be2-99ea-9e9fa7b0e6dc"
-      (reference "#PWR0116") (unit 1) (value "GND") (footprint "")
-    )
     (path "/d5462351-ea88-4cff-a4e2-2b958fc06bdb"
       (reference "#PWR0117") (unit 1) (value "GND") (footprint "")
@@
       (reference "D5") (unit 1) (value "LED_Small") (footprint "LED_SMD:LED_0805_2012Metric_Pad1.15x1.40mm_HandSolder")
     )
-    (path "/83035ccb-c0eb-4b44-b493-ac9a52db9015"
-      (reference "D6") (unit 1) (value "D_TVS") (footprint "Diode_SMD:D_SOD-323_HandSoldering")
-    )
-    (path "/7743cf6a-5b95-4f42-b28f-1967b554d759"
-      (reference "D7") (unit 1) (value "D_TVS") (footprint "Diode_SMD:D_SOD-323_HandSoldering")
-    )
     (path "/24adc8c0-9521-418c-a6a0-aa8f7fa285cd"
       (reference "J1") (unit 1) (value "TOP") (footprint "Footprints:RoundPinHeader_1x12")
@@
       (reference "SW2") (unit 1) (value "Power Switch") (footprint "Footprints:PTS636SK25SMTRLFS")
     )
-    (path "/fa997c01-e394-407e-9af2-b0b4d5648f4e"
-      (reference "SW3") (unit 1) (value "Config Switch") (footprint "Footprints:PTS636SK25SMTRLFS")
+    (path "/5b302fa4-059a-4878-8524-670aea735c7c"
+      (reference "SW?") (unit 1) (value "SW_DIP_x01") (footprint "")
     )
     (path "/bfaec5dd-dca1-4ce3-a1de-1f59bdc18b31"
