File: bm83-featherwing/bm83-featherwing.kicad_pcb (KiCad board)
At the start: 2 copper layers, 22.9 x 59.4 mm, 23 parts, among them J1 TOP, J2 BOT, J3 DX07S016JA1R1500, SW1 Reset Switch, SW2 Power Switch, SW3 SW_DIP_x01, U1 BM83SM1-00AA

Commit message: BM83 rev 2 ordered.
Other:
- board text added: "05/2021"
- board text added: "3V3"
- board text added: "BCK"
- board text added: "BM83 BLUETOOTH 5.0 AUDIO WING"
- board text added: "DO"
- board text added: "WS"
- board text removed: "+3V3"
- board text removed: "CK"
- board text removed: "DI"
- board text removed: "LR"
Changed lines of the file:
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@@
       (effects (font (size 1 1) (thickness 0.2)))
     )
-    (fp_text user "${REFERENCE}" (at 0 -1.524) (layer "F.SilkS")
+    (fp_text user "${REFERENCE}" (at -2.667 0 90) (layer "F.SilkS")
       (effects (font (size 1 1) (thickness 0.2)))
     )
@@
       (effects (font (size 1 1) (thickness 0.15)))
     )
-    (fp_text value "1uF" (at -3.556 0 90) (layer "F.SilkS")
+    (fp_text value "1uF" (at 2.54 0 180) (layer "F.SilkS")
       (effects (font (size 1 1) (thickness 0.2)))
     )
@@
       (effects (font (size 1 1) (thickness 0.2)))
     )
-    (fp_text user "${REFERENCE}" (at 0 1.524) (layer "F.SilkS")
+    (fp_text user "${REFERENCE}" (at -2.794 0 90) (layer "F.SilkS")
       (effects (font (size 1 1) (thickness 0.2)))
     )
@@
       (effects (font (size 1 1) (thickness 0.15)) (justify mirror))
     )
-    (fp_text value "1uF" (at 0 -1.68) (layer "B.Fab")
+    (fp_text value "1uF" (at 0 -1.68) (layer "B.SilkS")
       (effects (font (size 1 1) (thickness 0.2)) (justify mirror))
     )
@@
       (effects (font (size 1 1) (thickness 0.15)) (justify mirror))
     )
-    (fp_text value "0.1uF" (at 3.81 0 90) (layer "B.Fab")
+    (fp_text value "0.1uF" (at 4.318 0 90) (layer "B.SilkS")
       (effects (font (size 1 1) (thickness 0.2)) (justify mirror))
     )
@@
       (effects (font (size 1 1) (thickness 0.15)) (justify mirror))
     )
-    (fp_text value "4.7K" (at 0 -1.65) (layer "B.Fab")
+    (fp_text value "4.7K" (at 0 -1.65) (layer "B.SilkS")
       (effects (font (size 1 1) (thickness 0.2)) (justify mirror))
     )
@@
       (effects (font (size 1 1) (thickness 0.15)) (justify mirror))
     )
-    (fp_text value "5.1K" (at 0 -1.65 -270) (layer "B.Fab")
+    (fp_text value "5.1K" (at -3.556 0 -270) (layer "B.SilkS")
       (effects (font (size 1 1) (thickness 0.2)) (justify mirror))
     )
@@
       (effects (font (size 1 1) (thickness 0.15)) (justify mirror))
     )
-    (fp_text value "0.1uF" (at 3.81 0 90) (layer "B.Fab")
+    (fp_text value "0.1uF" (at 4.318 0 90) (layer "B.SilkS")
       (effects (font (size 1 1) (thickness 0.2)) (justify mirror))
     )
@@
       (effects (font (size 1 1) (thickness 0.15)) (justify mirror))
     )
-    (fp_text value "5.1K" (at 0 -1.65 90) (layer "B.Fab")
+    (fp_text value "5.1K" (at 3.572 0.016 90) (layer "B.SilkS")
       (effects (font (size 1 1) (thickness 0.2)) (justify mirror))
     )
@@
       (effects (font (size 1 1) (thickness 0.15)) (justify mirror))
     )
-    (fp_text value "SMBJ10CA" (at 0 -3) (layer "B.Fab")
+    (fp_text value "SMBJ10CA" (at 0 3.048) (layer "B.SilkS")
       (effects (font (size 1 1) (thickness 0.2)) (justify mirror))
     )
@@
     )
   )
+  (gr_line (start 153.924 114.935) (end 153.924 116.459) (layer "F.SilkS") (width 0.12))
+  (gr_line (start 138.684 117.983) (end 138.684 114.935) (layer "F.SilkS") (width 0.12))
+  (gr_line (start 147.32 116.459) (end 147.32 117.983) (layer "F.SilkS") (width 0.12))
+  (gr_line (start 147.32 117.983) (end 138.684 117.983) (layer "F.SilkS") (width 0.12))
+  (gr_line (start 138.684 114.935) (end 153.924 114.935) (layer "F.SilkS") (width 0.12))
+  (gr_line (start 153.924 116.459) (end 147.32 116.459) (layer "F.SilkS") (width 0.12))
   (gr_arc (start 141.732 128.778) (end 141.224 128.778) (angle -90) (layer "Edge.Cuts") (width 0.05))
   (gr_line (start 154.94 128.27) (end 151.892 128.27) (layer "Edge.Cuts") (width 0.05))
@@
   (gr_line (start 157.48 72.39) (end 157.48 125.73) (layer "Edge.Cuts") (width 0.05))
   (gr_line (start 134.62 125.73) (end 134.62 72.39) (layer "Edge.Cuts") (width 0.05))
-  (gr_text "+3V3" (at 154.813 119.38 270) (layer "F.SilkS")
-    (effects (font (size 0.9 0.9) (thickness 0.2)))
-  )
-  (gr_text "LR" (at 154.813 104.14 270) (layer "F.SilkS")
+  (gr_text "3V3" (at 154.813 119.38 -90) (layer "B.SilkS")
+    (effects (font (size 0.9 0.9) (thickness 0.2)) (justify mirror))
+  )
+  (gr_text "GND" (at 154.813 114.3 -90) (layer "B.SilkS")
+    (effects (font (size 0.9 0.9) (thickness 0.2)) (justify mirror))
+  )
+  (gr_text "WS" (at 154.813 104.14 90) (layer "F.SilkS")
     (effects (font (size 0.9 0.9) (thickness 0.2)))
   )
@@
     (effects (font (size 0.9 0.9) (thickness 0.2)))
   )
-  (gr_text "CK" (at 154.813 106.68 270) (layer "F.SilkS")
-    (effects (font (size 0.9 0.9) (thickness 0.2)))
-  )
-  (gr_text "MCK" (at 154.813 88.9 270) (layer "F.SilkS")
+  (gr_text "BCK" (at 154.813 106.68 90) (layer "F.SilkS")
+    (effects (font (size 0.9 0.9) (thickness 0.2)))
+  )
+  (gr_text "MCK" (at 154.813 88.9 90) (layer "F.SilkS")
     (effects (font (size 0.9 0.9) (thickness 0.2)))
   )
@@
     (effects (font (size 0.9 0.9) (thickness 0.2)))
   )
-  (gr_text "MFB" (at 137.287 101.6 90) (layer "F.SilkS")
-    (effects (font (size 0.9 0.9) (thickness 0.2)))
-  )
-  (gr_text "RX" (at 137.287 96.52 90) (layer "F.SilkS")
+  (gr_text "MFB" (at 137.287 101.6 270) (layer "F.SilkS")
+    (effects (font (size 0.9 0.9) (thickness 0.2)))
+  )
+  (gr_text "05/2021" (at 147.574 117.221) (layer "F.SilkS")
+    (effects (font (size 0.8 0.8) (thickness 0.15)) (justify left))
+  )
+  (gr_text "RX" (at 137.287 96.52 270) (layer "F.SilkS")
     (effects (font (size 0.9 0.9) (thickness 0.2)))
   )
@@
     (effects (font (size 0.9 0.9) (thickness 0.2)))
   )
-  (gr_text "TX" (at 137.287 99.06 90) (layer "F.SilkS")
-    (effects (font (size 0.9 0.9) (thickness 0.2)))
-  )
-  (gr_text "DI" (at 154.813 101.6 270) (layer "F.SilkS")
+  (gr_text "TX" (at 137.287 99.06 270) (layer "F.SilkS")
+    (effects (font (size 0.9 0.9) (thickness 0.2)))
+  )
+  (gr_text "DO" (at 154.813 101.6 90) (layer "F.SilkS")
     (effects (font (size 0.9 0.9) (thickness 0.2)))
   )
@@
     (effects (font (size 0.9 0.9) (thickness 0.2)))
   )
-  (gr_text "GND" (at 154.813 114.3 270) (layer "F.SilkS")
-    (effects (font (size 0.9 0.9) (thickness 0.2)))
+  (gr_text "BM83 BLUETOOTH 5.0\nAUDIO WING" (at 138.811 116.459) (layer "F.SilkS")
+    (effects (font (size 0.9 0.9) (thickness 0.2)) (justify left))
   )
   (segment (start 144.272 119.888) (end 143.022 119.888) (width 0.25) (layer "F.Cu") (net 1))
